File: breakout-board/kicad/bobcat-dash-breakout.kicad_pcb (KiCad board)
At the start: 2 copper layers, 150 x 134 mm, 143 parts, among them J1 TO PI (40-pin ribbon), J10 ADS1115, J11 LIGHTS, J12 COIL, J2 POWER IN, J3 TO 5V BUCK, J4 SWITCHES, J5 TACH, J6 FUEL, J7 HORN, J8 SILENCE, J9 MAX98357A, Q1 IRLZ44N, Q2 IRF4905, Q3 BC547B, Q4 BC547B, U1 PC817, U10 PC817, U4 PC817, U5 PC817, U6 CD4060BE, U7 PC817, U8 PC817, U9 PC817

Commit message: Machine angle display, safe tilt zeroing, board rev 2.6 (latching TILT connector)
Software:
- Machine angle panel: roll (rear view) and pitch (side view) skid steer outlines that tilt with
  the machine, with amber/red limits (roll 8/15 deg, nose up 15/20, nose down 20/25; not Bobcat
  figures). Battery and fuel share one panel; warning tiles shorter. [tilt] enabled = false restores
  the original layout.
- tilt.py: LSM6DSOX reader with gyro/accelerometer blending (bumps move it < 1 deg), start-up
  averaging so a restart on a slope reads the true angle at once, and --zero-tilt that refuses on a
  slope (> 5 deg) or while moving unless --force.
- Simulator: Left/Right roll, , / . pitch, 0 level.
- Light indicators back to the small icons by default (display = "tiles" still available).

Breakout board:
- rev 2.5: TILT connector J13 (GND, 3V3, SDA, SCL) with 100R SDA/SCL and 47R 3V3 protection.
- rev 2.6: J13 is a latching Molex Micro-Fit 3.0 (43650-0415). Harness stays Phoenix MSTB
  (14-16 AWG); README covers securing the plugs against vibration.
- Schematic block subtitles now wrap to fit their boxes.

Docs and BOM updated (tilt sensor, Micro-Fit housing and pins, sensor cable).

Co-Authored-By: Claude Opus 5.5 <noreply@anthropic.com>
Parts:
- added J13: TILT, Connector_Molex:Molex_Micro-Fit_3.0_43650-0415_1x04_P3.00mm_Vertical, F.Cu at (30.0, 4.40)
- added R83: 100, Resistor_THT:R_Axial_DIN0207_L6.3mm_D2.5mm_P7.62mm_Horizontal, F.Cu at (33.6, 10.6)
- added R84: 100, Resistor_THT:R_Axial_DIN0207_L6.3mm_D2.5mm_P7.62mm_Horizontal, F.Cu at (37.2, 10.6)
- added R85: 47, Resistor_THT:R_Axial_DIN0207_L6.3mm_D2.5mm_P7.62mm_Horizontal, F.Cu at (30.0, 10.6)
Routing:
- net SDA: track 77.1 -> 123.6 mm, vias 2 -> 0
- net +12V_IN: track 96.8 -> 142.9 mm
- net GND: track 963.4 -> 922.6 mm, vias 1 -> 0
- net +12V: track 390.1 -> 352.3 mm, vias 4 -> 1
- net SCL: track 70.3 -> 93.1 mm
- net +3V3: track 250.1 -> 269.2 mm, vias 0 -> 2
- net LT_REAR_GPIO: track 111.3 -> 127.9 mm, vias 0 -> 1
- net /TILT_3V3: track 0.00 -> 15.8 mm
- net HORN_G: track 144.4 -> 159.5 mm
- net /TILT_SDA: track 0.00 -> 14.8 mm
- net /TILT_SCL: track 0.00 -> 14.6 mm
- net BATT_ADC: track 107.8 -> 122.2 mm
- net +12V_HORN: track 144.8 -> 158.9 mm
- net HOLD_GPIO: track 247.1 -> 234.0 mm, vias 1 -> 2
- net BTN_GPIO: track 143.8 -> 131.8 mm
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Other:
- board text added: "TILT SENSOR (I2C)"
- board text added: "rev 2.6 2026-10"
- board text removed: "rev 2.4 2026-10"
